File: pcb/audio-amplifier/audio-amplifier.kicad_sch (KiCad schematic)
At the start: 0 parts

Commit message: pcb: Add PCB
Parts:
- added C1, C2, C4, C5, C6, C7, C8: 100nF, Capacitor_SMD:C_0805_2012Metric, symbol audio-amplifier:C_100nF_0805
- added C3: 27pF, Capacitor_SMD:C_0603_1608Metric, symbol audio-amplifier:C_27pF_0603_C0G
- added H1, H2, H3, H4: MountingHole_Pad, MountingHole:MountingHole_3.2mm_M3_Pad_Via, symbol Mechanical:MountingHole_Pad
- added J1: PJ-320D, Connector_Audio:Jack_3.5mm_PJ320D_Horizontal, symbol audio-amplifier:AudioJack4_PJ-320D
- added J2, J3, J4: WJ500V-5.08-2P, TerminalBlock:TerminalBlock_bornier-2_P5.08mm, symbol audio-amplifier:Screw_Terminal_01x02
- added R1, R2: 100R, Resistor_SMD:R_0805_2012Metric, symbol audio-amplifier:R_100R_0805
- added R10, R11, R14, R15, R22, R5, R6: 10K, Resistor_SMD:R_0805_2012Metric, symbol audio-amplifier:R_10K_0805
- added R12, R13, R9: 100K, Resistor_SMD:R_0805_2012Metric, symbol audio-amplifier:R_100K_0805
- added R3: 4K7, Resistor_SMD:R_0603_1608Metric, symbol audio-amplifier:R_4K7_0603_Thin_Film
- added R4: 100K, Resistor_SMD:R_0603_1608Metric, symbol audio-amplifier:R_100K_0603_Thin_Film
- added R7, R8: R, Resistor_SMD:R_0805_2012Metric, symbol audio-amplifier:R
- added U1: LMC555M, Package_SO:SOP-8_3.9x4.9mm_P1.27mm, symbol audio-amplifier:Timer_LMC555M
- added U2, U3, U4: COS2353SR, Package_SO:SOP-8_3.9x4.9mm_P1.27mm, symbol audio-amplifier:Amplifier_Operational_COS2353SR
- added U5, U6: TLV3201, Package_TO_SOT_SMD:SOT-23-5, symbol audio-amplifier:Comparator_TLV3201
Connections:
- new net: R7.2, R8.1, R9.1, U2.2 (-)
- new net: C2.2, R12.1, R5.2, R6.1, U3.3 (+)
- new net: C2.1, R1.2, R2.2
- new net: U4.6 (-), U4.7, U5.4 (-)
- new net: U3.1, U3.2 (-), U6.4 (-)
- new net: R10.2, R11.1, R13.1, U4.3 (+)
- new net: R13.2, U4.1, U4.5 (+)
- new net: C3.1, R4.2, U1.2 (TR), U1.6 (THR), U2.3 (+)
- new net: R22.2, U1.4 (R)
- new net: R3.2, R4.1, U1.7 (DIS)
- new net: J1.T, R2.1
- new net: R12.2, U4.2 (-)
- new net: J1.R1, R1.1
- new net +10V: J3.2 (Pin_2), R14.1, R15.1
- new net +5V: C1.1, C4.1, C5.1, C6.1, C7.1, C8.1, J2.2 (Pin_2), R10.1, R22.1, R3.1, R5.1, R7.1, U1.8 (VCC), U2.8 (V+), U3.8 (V+), U4.8 (V+), U5.5 (V+), U6.5 (V+)
- new net GND: C1.2, C3.2, C4.2, C5.2, C6.2, C7.2, C8.2, H1.1, H2.1, H3.1, H4.1, J1.R2, J1.S, J2.1 (Pin_1), J3.1 (Pin_1), R11.2, R6.2, R8.2, U1.1 (GND), U2.4 (V-), U3.4 (V-), U4.4 (V-), U5.2 (GND), U6.2 (GND)
- new net Half Bridge Driver Left/EN: R14.2
- new net Half Bridge Driver Left/PWM: U5.1
- new net Half Bridge Driver Right/EN: R15.2
- new net Half Bridge Driver Right/PWM: U6.1
- new net OUT+: J4.1 (Pin_1)
- new net OUT-: J4.2 (Pin_2)
- new net TRIANGLE: R9.2, U2.1, U5.3 (+), U6.3 (+)
- no-connect marks 0 -> 8
Other:
- added sheet Half Bridge Driver Left (half-bridge-driver.kicad_sch)
- added sheet Half Bridge Driver Right (half-bridge-driver.kicad_sch)
- added sheet Low Pass Filter (low-pass-filter.kicad_sch)
- note added: "2 half bridges forming a full bridge."
- note added: "Add DC offset to AC signal"
- note added: "Audio out connector"
- note added: "Inverting audio signal"
- note added: "PWM modulation for audio signal"
- note added: "Simple stereo to mono conversion"
- note added: "Triangle wave generator"
- note added: "~240 KHz triangle wave generator"

Commit message: Add updated PCB
Parts:
- removed R7, R8: R, Resistor_SMD:R_0805_2012Metric, symbol audio-amplifier:R
- added C26: 330nF, Capacitor_SMD:C_0805_2012Metric, symbol audio-amplifier:C_330nF_0805
- added C27: 100nF, Capacitor_SMD:C_0805_2012Metric, symbol audio-amplifier:C_100nF_0805
- added C28: 4.7uF, Capacitor_SMD:C_1206_3216Metric, symbol audio-amplifier:C_4.7uF_1206
- added D1: SS54, Diode_SMD:D_SMA_Handsoldering, symbol audio-amplifier:D_SS54
- added R23, R24: 50R, Resistor_SMD:R_0805_2012Metric, symbol audio-amplifier:R_50R_0805
- added R7, R8: 226K, Resistor_SMD:R_0805_2012Metric, symbol audio-amplifier:R_226K_0805
- added U11: LDO_L78M05CDT_SOT89, Package_TO_SOT_SMD:TO-252-2, symbol audio-amplifier:LDO_L78M05CDT_SOT89
- renumbered U3 to U2, U2 to U3
Connections:
- net +10V: now also C26.1, D1.1 (K), U11.1 (IN)
- net +5V: now also C27.1, C28.1, D1.2 (A), R7.1, U11.3 (OUT)
- net GND: now also C26.2, C27.2, C28.2, R8.2, U11.2 (GND)
- net Half Bridge Driver Left/PWM: now also R23.2; no longer U5.1
- net Half Bridge Driver Right/PWM: now also R24.2; no longer U6.1
- net at R9.1, U2.2 (-): now also R7.2, R8.1
- new net: R23.1, U5.1
- new net: R24.1, U6.1
