File: pcb/audio-amplifier/half-bridge-driver.kicad_sch (KiCad schematic)
At the start: 12 parts, among them Q1 IRFR4615TRLPBF, Q2 IRFR4615TRLPBF, U7 74LVC1G04SE, U8 DGD05473

Commit message: Add updated PCB
Parts:
- added R25: 50R, Resistor_SMD:R_0805_2012Metric, symbol audio-amplifier:R_50R_0805
Connections:
- net VCC: no longer C?.1, U7.5 (VCC)
- net at U7.4: now also R25.1; no longer U8.8 (LIN)
- new net: R25.2, U8.8 (LIN)
- new net +5V: C?.1, U7.5 (VCC)
Changed lines of the file:
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@@
+    (stroke (width 0) (type default))
+  )
+  (wire (pts (xy 86.36 100.33) (xy 87.63 100.33))
     (stroke (width 0) (type default))
   )
@@
   )
   (wire (pts (xy 130.81 93.98) (xy 130.81 90.17))
-    (stroke (width 0) (type default))
-  )
-  (wire (pts (xy 86.36 100.33) (xy 109.22 100.33))
     (stroke (width 0) (type default))
   )
@@
   )
   (wire (pts (xy 72.39 109.22) (xy 72.39 110.49))
+    (stroke (width 0) (type default))
+  )
+  (wire (pts (xy 95.25 100.33) (xy 109.22 100.33))
     (stroke (width 0) (type default))
   )
@@
     (effects (font (size 1.27 1.27)) (justify left))
   )
-  (hierarchical_label "VCC" (shape input) (at 72.39 80.01 90) (fields_autoplaced)
-    (effects (font (size 1.27 1.27)) (justify left))
+  (netclass_flag "" (length 2.54) (shape round) (at 96.52 100.33 180) (fields_autoplaced)
+    (effects (font (size 1.27 1.27)) (justify right bottom))
+    (property "Netclass" "50ohm" (at 97.2185 102.87 0)
+      (effects (font (size 1.27 1.27) italic) (justify left))
+    )
+  )
+  (netclass_flag "" (length 2.54) (shape round) (at 87.63 100.33 180) (fields_autoplaced)
+    (effects (font (size 1.27 1.27)) (justify right bottom))
+    (property "Netclass" "50ohm" (at 88.3285 102.87 0)
+      (effects (font (size 1.27 1.27) italic) (justify left))
+    )
   )
   (symbol (lib_id "audio-amplifier:C_4.7uF_1206") (at 86.36 43.18 0) (unit 1)
@@
       (effects (font (size 1.27 1.27)) hide)
     )
+    (pin "1")
     (pin "2")
     (pin "3")
@@
         (path "/181bc403-0d49-4b2a-87e2-cf403d77be4c/a96eaf2c-e309-4807-b2ee-df2dcf4e128c"
           (reference "R19") (unit 1)
+        )
+      )
+    )
+  )
+  (symbol (lib_id "power:+5V") (at 72.39 80.01 0) (unit 1)
+    (in_bom yes) (on_board yes) (dnp no) (fields_autoplaced)
+    (property "Reference" "#PWR053" (at 72.39 83.82 0)
+      (effects (font (size 1.27 1.27)) hide)
+    )
+    (property "Value" "+5V" (at 72.39 76.2 0)
+      (effects (font (size 1.27 1.27)))
+    )
+    (property "Footprint" "" (at 72.39 80.01 0)
+      (effects (font (size 1.27 1.27)) hide)
+    )
+    (property "Datasheet" "" (at 72.39 80.01 0)
+      (effects (font (size 1.27 1.27)) hide)
+    )
+    (pin "1")
+    (instances
+      (project "audio-amplifier"
+        (path "/181bc403-0d49-4b2a-87e2-cf403d77be4c/e00e7b8a-da56-4912-897b-c38236cda570"
+          (reference "#PWR053") (unit 1)
+        )
+        (path "/181bc403-0d49-4b2a-87e2-cf403d77be4c/a96eaf2c-e309-4807-b2ee-df2dcf4e128c"
+          (reference "#PWR054") (unit 1)
         )
       )
@@
         )
       )
+    )
+  )
+  (symbol (lib_id "audio-amplifier:R_50R_0805") (at 91.44 100.33 90) (unit 1)
+    (in_bom yes) (on_board yes) (dnp no) (fields_autoplaced)
+    (property "Reference" "R25" (at 91.44 95.25 90)
+      (effects (font (size 1.27 1.27)))
+    )
+    (property "Value" "50R" (at 91.44 97.79 90)
+      (effects (font (size 1.27 1.27)))
+    )
+    (property "Footprint" "Resistor_SMD:R_0805_2012Metric" (at 91.44 102.108 90)
+      (effects (font (size 1.27 1.27)) hide)
+    )
+    (property "Datasheet" "https://datasheet.lcsc.com/lcsc/2105241808_Viking-Tech-ARG05FTC0500_C2828866.pdf" (at 91.44 100.33 0)
+      (effects (font (size 1.27 1.27)) hide)
+    )
+    (property "LCSC Part #" "C2828866" (at 91.44 100.33 0)
+      (effects (font (size 1.27 1.27)) hide)
+    )
+    (property "MPN" "ARG05FTC0500" (at 91.44 100.33 0)
+      (effects (font (size 1.27 1.27)) hide)
+    )
+    (pin "1")
+    (pin "2")
+    (instances
+      (project "audio-amplifier"
+        (path "/181bc403-0d49-4b2a-87e2-cf403d77be4c/e00e7b8a-da56-4912-897b-c38236cda570"
+          (reference "R25") (unit 1)
+        )
+        (path "/181bc403-0d49-4b2a-87e2-cf403d77be4c/a96eaf2c-e309-4807-b2ee-df2dcf4e128c"
+          (reference "R26") (unit 1)
+        )
+      )
